File: Polarimeter.kicad_sch (KiCad schematic)
At the start: 39 parts, among them IC1 ADS8355IRTET, J1 Conn_02x24_Counter_Clockwise, U1 OPA2320AID, U2 OPA381AIDRBT, U3 OPA381AIDRBT, U4 REF3425IDBVR, U5 OPA320AIDBVR, U6 OPA320AIDBVR

Commit message: Add rendered docs, clean up sheet naming
- Export schematic PDF and top/bottom 3D board renders to docs/
- Embed renders + schematic PDF link in README
- Rename hierarchical sub-sheet untitled.kicad_sch -> Power.kicad_sch
  and update references in root schematic and PCB
- Remove stale orphaned duplicate of the power sheet
- Credit co-designer

Co-Authored-By: Claude Opus 4.8 <noreply@anthropic.com>
Other:
- sheet power: file untitled.kicad_sch -> Power.kicad_sch
Changed lines of the file:
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@@
 			)
 		)
-		(property "Sheetfile" "untitled.kicad_sch"
+		(property "Sheetfile" "Power.kicad_sch"
 			(at 332.74 62.8146 0)
 			(effects
