File: Power.kicad_sch (KiCad schematic)
At the start: 25 parts, among them J2 PJ-037AH, SW1 TS01CQE, U7 LT8609EMSE-TRPBF, U8 LP5912-3.3DRV, U9 ADR130AUJZ-REEL7

Commit message: Add rendered docs, clean up sheet naming
- Export schematic PDF and top/bottom 3D board renders to docs/
- Embed renders + schematic PDF link in README
- Rename hierarchical sub-sheet untitled.kicad_sch -> Power.kicad_sch
  and update references in root schematic and PCB
- Remove stale orphaned duplicate of the power sheet
- Credit co-designer

Co-Authored-By: Claude Opus 4.8 <noreply@anthropic.com>
Parts:
- C14: footprint (none) -> Capacitor_SMD:C_2220_5750Metric
- C15, C19, C22, C24: footprint (none) -> Capacitor_SMD:C_0805_2012Metric
- C16, C17, C18, C20, C21, C23, C26, C27: footprint (none) -> Capacitor_SMD:C_0603_1608Metric
- C25: value 10u -> v; footprint (none) -> Capacitor_SMD:C_0805_2012Metric
- J2: footprint CONN_37AH -> PJ-037AH:CONN_37AH
- L1: footprint (none) -> Inductor_SMD:L_Coilcraft_XxL4020
- R12, R13, R14, R16: footprint (none) -> Resistor_SMD:R_0603_1608Metric; symbol Device:R -> Device:R_US
- R15: value 187 k -> 187k; footprint (none) -> Resistor_SMD:R_0603_1608Metric; symbol Device:R -> Device:R_US
- SW1: footprint TS01CQE_CNK -> TS01CQE:TS01CQE_CNK
- U7: footprint 05-08-1664_ADI -> LT8609EMSE-TRPBF:05-08-1664_ADI
- U9: footprint UJ_6_ADI -> ADR130AUJZ-REEL7:UJ_6_ADI
Changed lines of the file:
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@@
 	)
 	(symbol
-		(lib_id "Device:R")
+		(lib_id "Device:R_US")
 		(at 74.93 93.98 0)
 		(mirror x)
@@
 			)
 		)
-		(property "Footprint" ""
+		(property "Footprint" "Resistor_SMD:R_0603_1608Metric"
 			(at 73.152 93.98 90)
 			(effects
@@
 			)
 		)
-		(property "Description" "Resistor"
+		(property "Description" "Resistor, US symbol"
 			(at 74.93 93.98 0)
 			(effects
@@
 			)
 		)
-		(property "Footprint" "05-08-1664_ADI"
+		(property "Footprint" "LT8609EMSE-TRPBF:05-08-1664_ADI"
 			(at 41.91 55.88 0)
 			(effects
@@
 			)
 		)
-		(property "Footprint" ""
+		(property "Footprint" "Capacitor_SMD:C_0603_1608Metric"
 			(at 101.6 65.0748 0)
 			(effects
@@
 			)
 		)
-		(property "Footprint" ""
+		(property "Footprint" "Capacitor_SMD:C_0603_1608Metric"
 			(at 210.5152 80.01 0)
 			(effects
@@
 			)
 		)
-		(property "Footprint" "UJ_6_ADI"
+		(property "Footprint" "ADR130AUJZ-REEL7:UJ_6_ADI"
 			(at 208.28 67.31 0)
 			(effects
@@
 			)
 		)
-		(property "Footprint" ""
+		(property "Footprint" "Capacitor_SMD:C_2220_5750Metric"
 			(at 184.4548 29.21 0)
 			(effects
@@
 			)
 		)
-		(property "Footprint" ""
+		(property "Footprint" "Capacitor_SMD:C_0603_1608Metric"
 			(at 143.8148 29.21 0)
 			(effects
@@
 	)
 	(symbol
-		(lib_id "Device:R")
+		(lib_id "Device:R_US")
 		(at 74.93 101.6 0)
 		(mirror x)
@@
 			)
 		)
-		(property "Value" "187 k"
+		(property "Value" "187k"
 			(at 78.74 101.6 90)
 			(effects
@@
 			)
 		)
-		(property "Footprint" ""
+		(property "Footprint" "Resistor_SMD:R_0603_1608Metric"
 			(at 73.152 101.6 90)
 			(effects
@@
 			)
 		)
-		(property "Description" "Resistor"
+		(property "Description" "Resistor, US symbol"
 			(at 74.93 101.6 0)
 			(effects
@@
 			)
 		)
-		(property "Footprint" ""
+		(property "Footprint" "Capacitor_SMD:C_0805_2012Metric"
 			(at 59.3852 90.17 0)
 			(effects
@@
 			)
 		)
-		(property "Footprint" ""
+		(property "Footprint" "Inductor_SMD:L_Coilcraft_XxL4020"
 			(at 50.8 90.17 0)
 			(effects
@@
 			)
 		)
-		(property "Footprint" ""
+		(property "Footprint" "Capacitor_SMD:C_0805_2012Metric"
 			(at 150.8252 59.69 0)
 			(effects
@@
 			)
 		)
-		(property "Footprint" ""
+		(property "Footprint" "Capacitor_SMD:C_0603_1608Metric"
 			(at 265.1252 80.01 0)
 			(effects
@@
 			)
 		)
-		(property "Value" "10u"
+		(property "Value" "v"
 			(at 173.99 64.7699 0)
 			(effects
@@
 			)
 		)
-		(property "Footprint" ""
+		(property "Footprint" "Capacitor_SMD:C_0805_2012Metric"
 			(at 171.1452 67.31 0)
 			(effects
@@
 			)
 		)
-		(property "Footprint" ""
+		(property "Footprint" "Capacitor_SMD:C_0603_1608Metric"
 			(at 157.7848 29.21 0)
 			(effects
@@
 			)
 		)
-		(property "Footprint" ""
+		(property "Footprint" "Capacitor_SMD:C_0603_1608Metric"
 			(at 128.5748 29.21 0)
 			(effects
@@
 			)
 		)
-		(property "Footprint" "CONN_37AH"
+		(property "Footprint" "PJ-037AH:CONN_37AH"
 			(at 27.94 20.32 0)
 			(effects
@@
 	)
 	(symbol
-		(lib_id "Device:R")
+		(lib_id "Device:R_US")
 		(at 33.02 66.04 90)
 		(mirror x)
@@
 			)
 		)
-		(property "Footprint" ""
+		(property "Footprint" "Resistor_SMD:R_0603_1608Metric"
 			(at 33.02 64.262 90)
 			(effects
@@
 			)
 		)
-		(property "Description" "Resistor"
+		(property "Description" "Resistor, US symbol"
 			(at 33.02 66.04 0)
 			(effects
@@
 	)
 	(symbol
-		(lib_id "Device:R")
+		(lib_id "Device:R_US")
 		(at 55.88 93.98 0)
 		(mirror x)
@@
 			)
 		)
-		(property "Footprint" ""
+		(property "Footprint" "Resistor_SMD:R_0603_1608Metric"
 			(at 54.102 93.98 90)
 			(effects
@@
 			)
 		)
-		(property "Description" "Resistor"
+		(property "Description" "Resistor, US symbol"
 			(at 55.88 93.98 0)
 			(effects
@@
 			)
 		)
-		(property "Footprint" ""
+		(property "Footprint" "Capacitor_SMD:C_0603_1608Metric"
 			(at 36.83 59.9948 0)
 			(effects
@@
 			)
 		)
-		(property "Footprint" ""
+		(property "Footprint" "Capacitor_SMD:C_0805_2012Metric"
 			(at 170.4848 29.21 0)
 			(effects
@@
 			)
 		)
-		(property "Footprint" ""
+		(property "Footprint" "Capacitor_SMD:C_0805_2012Metric"
 			(at 92.71 61.9252 0)
 			(effects
@@
 			)
 		)
-		(property "Footprint" ""
+		(property "Footprint" "Capacitor_SMD:C_0603_1608Metric"
 			(at 68.2752 97.79 0)
 			(effects
@@
 	)
 	(symbol
-		(lib_id "Device:R")
+		(lib_id "Device:R_US")
 		(at 173.99 72.39 90)
 		(mirror x)
@@
 			)
 		)
-		(property "Footprint" ""
+		(property "Footprint" "Resistor_SMD:R_0603_1608Metric"
 			(at 173.99 70.612 90)
 			(effects
@@
 			)
 		)
-		(property "Description" "Resistor"
+		(property "Description" "Resistor, US symbol"
 			(at 173.99 72.39 0)
 			(effects
@@
 			)
 		)
-		(property "Footprint" "TS01CQE_CNK"
+		(property "Footprint" "TS01CQE:TS01CQE_CNK"
 			(at 96.52 22.86 0)
 			(effects
